File: OpenDrone_Transmitter_F103_HW.kicad_pcb (KiCad board)
At the start: 2 copper layers, 52 x 32 mm, 75 parts, among them J1 Conn_01x03, J10 Conn_01x04, J11 Conn_01x03, J12 Conn_01x04, J13 Conn_01x02, J14 Conn_01x05, J15 Conn_01x02, J16 Conn_02x04_Odd_Even, J17 Conn_01x02, J18 Conn_01x02, J19 Conn_01x03, J2 Conn_01x05, J20 Conn_01x02, J21 Conn_01x02, J22 Conn_01x02, J3 Conn_01x03, J4 Conn_01x03, J5 Conn_01x03, J6 Conn_01x02, J7 Conn_01x02, J8 Conn_01x03, J9 Conn_01x03, SW1 RESET, U1 STM32F103C8Tx, U2 AMS1117-3.3, U3 TPS54331, Y2 Crystal_GND24

Commit message: update project
Parts:
- added D4: SS24, Diode_SMD:D_SMA, F.Cu at (182.9, 100.2)
- J10, J12: footprint Footprint:Connector_XH_1x04_P1.25mm_Horizontal -> Footprint:Connector_XH_1x04_P1.25mm_Vertical
- J14, J2: footprint Footprint:Connector_XH_1x05_P1.25mm_Horizontal -> Footprint:Connector_XH_1x05_P1.25mm_Vertical
- moved C20 24.0 mm to (177.6, 92.2)
- moved C9 17.7 mm to (180.8, 92.2), turned to 90 degrees
- moved J2 7.06 mm to (219.3, 91.8)
- moved C12 6.90 mm to (172.8, 102.5), turned to 90 degrees
- moved SW1 5.01 mm to (217.6, 100.4)
- moved J19 4.88 mm to (216.8, 86.0)
- moved J4 4.88 mm to (219.3, 86.0)
- moved J14 4.74 mm to (212.1, 107.9)
- moved J10 4.63 mm to (203.2, 107.9)
- moved J12 4.63 mm to (195.4, 107.9)
- moved C17 4.19 mm to (210.6, 91.7)
- moved C29 4.19 mm to (210.6, 93.2)
- moved R15 4.19 mm to (210.6, 96.2)
- moved C15 4.19 mm to (210.6, 97.7)
- moved C19 4.19 mm to (210.6, 90.2)
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Other:
- board size 52 x 32 mm -> 57 x 32 mm

Commit message: update project
Parts:
- R1: value TBD -> 10k
- R2: value TBD -> 3,3k
- R6: value TBD -> 0R
- U3: footprint Package_SO:SOIC-8-1EP_3.9x4.9mm_P1.27mm_EP2.29x3mm_ThermalVias -> Package_SO:SOIC-8-1EP_3.9x4.9mm_P1.27mm_EP2.29x3mm
- moved J4 52.0 mm to (167.4, 88.5), turned to 90 degrees
- moved J5 49.4 mm to (216.7, 86.0), turned to -90 degrees
- moved C6 22.1 mm to (192.8, 86.1), turned to 90 degrees
- moved R3 21.9 mm to (194.3, 86.1), turned to -90 degrees
- moved C16 9.55 mm to (195.6, 104.2), turned to -90 degrees
- moved R11 7.48 mm to (190.2, 93.3)
- moved R12 7.48 mm to (190.2, 90.3)
- moved C26 7.48 mm to (190.2, 91.8)
- moved R7 5.62 mm to (190.3, 102.2), turned to 0 degrees
- moved C22 5.15 mm to (190.3, 100.7), turned to 180 degrees
- moved C28 4.52 mm to (190.2, 94.8)
- moved R14 4.52 mm to (190.2, 96.3)
- moved C27 4.48 mm to (190.3, 99.2)
- moved R13 4.48 mm to (190.3, 97.8)
- moved R1 3.26 mm to (179.0, 96.4)
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Connections:
- J3 pad 1: unconnected-(J3-Pin_1-Pad1) -> +3V3
- J3 pad 2: unconnected-(J3-Pin_2-Pad2) -> LEFT_JOYSTICK_IN1
- J3 pad 3: unconnected-(J3-Pin_3-Pad3) -> GND
- R1 pad 2: Net-(U3-VSENSE) -> Net-(R1-Pad2)
- R2 pad 1: Net-(R2-Pad1) -> Net-(U3-VSENSE)
- R6 pad 1: Net-(U3-VSENSE) -> Net-(R1-Pad2)
- R6 pad 2: Net-(R2-Pad1) -> Net-(U3-VSENSE)
Routing:
- net LEFT_JOYSTICK_IN1: track 0.00 -> 38.0 mm, vias 0 -> 1
- net LEFT_JOYSTICK_IN2: track 0.00 -> 33.0 mm, vias 0 -> 1
- net RIGHT_JOYSTICK_IN1: track 0.00 -> 27.3 mm, vias 0 -> 1
- net RIGHT_JOYSTICK_IN2: track 0.00 -> 23.0 mm, vias 0 -> 1
- net VOLUME_1: track 0.00 -> 20.9 mm
- net VOLUME_3: track 0.00 -> 19.3 mm
- net +3V3: track 0.00 -> 14.2 mm
- net STM32_RESET: track 0.00 -> 10.8 mm, vias 0 -> 2
- net OSC_IN: track 0.00 -> 9.09 mm
- net SENS_VOL: track 0.00 -> 8.99 mm
- net Net-(U3-BOOT): track 0.00 -> 8.84 mm, vias 0 -> 2
- net BUTTON1: track 0.00 -> 8.08 mm
- net SWITCH4: track 0.00 -> 7.40 mm
- net SWITCH2: track 0.00 -> 7.04 mm
- net SWITCH3: track 0.00 -> 7.02 mm
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- added copper zone on F.Cu, net +3V3
- added copper zone on F.Cu, net +5V
- added copper zone on B.Cu, net GND
- added copper zone on F.Cu, net GND
- added copper zone on F.Cu, net Net-(D1-K)
- added copper zone on F.Cu, net Net-(D2-A)
- added copper zone on F.Cu, net VBAT

Commit message: complete v1.0
Parts:
- added D5: D_Small, LED_SMD:LED_0603_1608Metric, F.Cu at (182.4, 85.2)
- added R17: 330R, Resistor_SMD:R_0603_1608Metric, F.Cu at (182.4, 88.2)
- moved C3 15.8 mm to (211.0, 90.7), turned to 0 degrees
- moved J14 15.7 mm to (196.4, 107.9)
- moved C6 10.9 mm to (203.8, 85.9)
- moved R3 10.9 mm to (205.3, 85.9)
- moved J12 8.91 mm to (204.4, 107.9)
- moved J10 8.85 mm to (212.0, 107.9)
- moved C16 6.35 mm to (190.2, 100.8), turned to 180 degrees
- moved R7 5.93 mm to (195.9, 104.1), turned to 90 degrees
- moved C22 5.33 mm to (194.4, 104.1), turned to -90 degrees
- moved C7 2.31 mm to (195.0, 85.9)
- moved R4 2.31 mm to (202.3, 85.9)
- moved C8 2.31 mm to (200.7, 85.9)
- moved Y2 2.31 mm to (197.9, 85.8)
- moved C15 2.04 mm to (211.0, 99.7)
- moved C17 2.04 mm to (211.0, 93.7)
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Connections:
- J14 pad 1: BUTTON1 -> BUTTON4
- J14 pad 2: BUTTON2 -> BUTTON3
- J14 pad 3: BUTTON3 -> BUTTON2
- J14 pad 4: BUTTON4 -> BUTTON1
- J16 pad 1: GND -> +3V3
- J16 pad 2: +3V3 -> GND
- J16 pad 3: NRF24_CE -> NRF24_CS
- J16 pad 4: NRF24_CS -> NRF24_CE
- J16 pad 5: NRF24_CLK -> NRF24_MOSI
- J16 pad 6: NRF24_MOSI -> NRF24_CLK
- J16 pad 7: NRF24_MISO -> NRF24_IRQ
- J16 pad 8: NRF24_IRQ -> NRF24_MISO
- J2 pad 3: STM32_CLK -> STM32_DIO
- J2 pad 4: STM32_DIO -> STM32_CLK
- U1 pad 19: ADC_RESERVED -> unconnected-(U1-PB1-Pad19)
- U1 pad 22: BUTTON1 -> NRF24_IRQ
- U1 pad 30: NRF24_IRQ -> BUTTON1
Routing:
- net +3V3: track 14.2 -> 205.0 mm, vias 0 -> 4
- net 5V_DEBUGGER: track 0.00 -> 56.7 mm, vias 0 -> 4
- net +5V: track 0.00 -> 49.4 mm
- net STM32_RESET: track 10.8 -> 41.7 mm
- net SWITCH1: track 6.65 -> 36.7 mm, vias 0 -> 2
- net SWITCH3: track 7.02 -> 35.5 mm, vias 0 -> 2
- net NRF24_MOSI: track 0.00 -> 27.3 mm, vias 0 -> 1
- net NRF24_CE: track 0.00 -> 26.1 mm, vias 0 -> 1
- net NRF24_CS: track 0.00 -> 25.4 mm, vias 0 -> 1
- net SWITCH2: track 7.04 -> 32.3 mm, vias 0 -> 1
- net VOLUME_2: track 0.00 -> 25.1 mm, vias 0 -> 1
- net VOLUME_4: track 0.00 -> 24.5 mm, vias 0 -> 1
- net STM32_DIO: track 0.00 -> 24.3 mm, vias 0 -> 1
- net NRF24_IRQ: track 0.00 -> 21.2 mm, vias 0 -> 1
- net SWITCH4: track 7.40 -> 28.2 mm, vias 0 -> 1
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Other:
- board text added: "3V3"
- board text added: "5V"
- board text added: "BT1"
- board text added: "BT2"
- board text added: "BT3"
- board text added: "BT4"
- board text added: "CE"
- board text added: "CLK"
- board text added: "CS"
- board text added: "DIO"
- board text added: "GND"
- board text added: "IRQ"
- board text added: "LIN1"
- board text added: "LIN2"
- board text added: "MISO"
- board text added: "MOSI"
- board text added: "OpenDrone Transmitter_F103_HW V1.0 Github: phonght32"
- board text added: "RIN1"
- board text added: "RIN2"
- board text added: "RST"
- board text added: "RX1"
- board text added: "SCL1"
- board text added: "SDA1"
- board text added: "SW1"
- board text added: "SW2"
- board text added: "SW3"
- board text added: "SW4"
- board text added: "TX1"
- board text added: "VBAT"
- board text added: "VOL1"
- board text added: "VOL2"
- board text added: "VOL3"
- board text added: "VOL4"

Commit message: update
Parts:
- added C10: 100nF, KiCad-Lib:C_0603_1608Metric, F.Cu at (193.1, 102.7)
- added C21: 100nF, KiCad-Lib:C_0603_1608Metric, F.Cu at (210.6, 99.8)
- added C30: 100nF, KiCad-Lib:C_0603_1608Metric, F.Cu at (190.1, 91.5)
- added C31: 100nF, KiCad-Lib:C_0603_1608Metric, F.Cu at (205.4, 84.7)
- added J23: Conn_01x08, KiCad-Lib:Connector_ZH_1x08_P1.25mm_Vertical, F.Cu at (198.9, 73.7)
- added R18: 1k, KiCad-Lib:R_0603_1608Metric, F.Cu at (194.6, 102.7)
- added R19: 1k, KiCad-Lib:R_0603_1608Metric, F.Cu at (210.6, 98.3)
- added R20: 1k, KiCad-Lib:R_0603_1608Metric, F.Cu at (190.1, 93.1)
- added R21: 1k, KiCad-Lib:R_0603_1608Metric, F.Cu at (206.9, 84.7)
- C1, C2, C20, C4, C5, C9: footprint Capacitor_SMD:C_1210_3225Metric -> KiCad-Lib:C_1210_3225Metric
- C11, C12, C13, C14, C15, C16, C17, C18, C19, C22, C23, C24, C25, C26, C27, C28, C29, C3, C6, C7, C8: footprint Capacitor_SMD:C_0603_1608Metric -> KiCad-Lib:C_0603_1608Metric
- D1, D2, D3, D4: footprint Diode_SMD:D_SMA -> KiCad-Lib:D_SMA
- D5: footprint LED_SMD:LED_0603_1608Metric -> KiCad-Lib:LED_0603_1608Metric
- J1, J11, J19, J3, J4, J5, J8, J9: footprint Footprint:Connector_XH_1x03_P1.25mm_Vertical -> KiCad-Lib:Connector_ZH_1x03_P1.25mm_Vertical
- J10, J12: footprint Footprint:Connector_XH_1x04_P1.25mm_Vertical -> KiCad-Lib:Connector_ZH_1x04_P1.25mm_Vertical
- J13, J15, J17, J18, J20, J21, J22, J6: footprint Footprint:Connector_XH_1x02_P1.25mm_Vertical -> KiCad-Lib:Connector_ZH_1x02_P1.25mm_Vertical
- J14, J2: footprint Footprint:Connector_XH_1x05_P1.25mm_Vertical -> KiCad-Lib:Connector_ZH_1x05_P1.25mm_Vertical
- J7: footprint Connector_JST:JST_EH_B2B-EH-A_1x02_P2.50mm_Vertical -> KiCad-Lib:Connector_ZH_1x02_P1.25mm_Vertical
- L1: footprint Footprint:Inductor_SMD_4D28 -> KiCad-Lib:Inductor_SMD_4D28
- R1, R10, R11, R12, R13, R14, R15, R16, R17, R2, R3, R4, R5, R6, R7, R8, R9: footprint Resistor_SMD:R_0603_1608Metric -> KiCad-Lib:R_0603_1608Metric
- SW1: footprint Footprint:Button_SMD_4.2x3.3x2.5mm -> KiCad-Lib:Button_SMD_4.2x3.3x2.5mm
- U3: footprint Package_SO:SOIC-8-1EP_3.9x4.9mm_P1.27mm_EP2.29x3mm -> KiCad-Lib:SOIC-8-1EP_3.9x4.9mm_P1.27mm_EP2.29x3mm
- U4: footprint Footprint:Board -> Proj-Lib:Board
- Y2: footprint Crystal:Crystal_SMD_3225-4Pin_3.2x2.5mm -> KiCad-Lib:Crystal_SMD_3225-4Pin_3.2x2.5mm
- moved C3 18.2 mm to (193.8, 84.8), turned to 90 degrees
- moved J2 17.5 mm to (211.4, 107.5), turned to 0 degrees
- moved SW1 12.0 mm to (222.2, 89.3)
- moved J15 11.3 mm to (215.4, 73.8), turned to 180 degrees
- moved R3 10.0 mm to (195.3, 84.8), turned to 90 degrees
- moved R4 9.75 mm to (210.6, 90.9), turned to 180 degrees
- moved J14 9.06 mm to (187.3, 107.5), turned to 0 degrees
- moved J18 8.90 mm to (210.3, 73.7), turned to 180 degrees
- moved J10 8.24 mm to (203.8, 107.5), turned to 0 degrees
- moved J6 8.23 mm to (179.9, 73.7), turned to 180 degrees
- moved J12 8.22 mm to (196.2, 107.5), turned to 0 degrees
- moved J17 7.74 mm to (174.8, 73.8), turned to 180 degrees
- moved J1 7.55 mm to (205.2, 73.7), turned to 180 degrees
- moved J20 7.47 mm to (179.9, 77.8), turned to 180 degrees
- moved C6 7.08 mm to (196.8, 84.8)
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Connections:
- net SWITCH1 renamed PB2
- net SWITCH2 renamed PB4
- net SWITCH3 renamed PB10
- net SWITCH4 renamed PB5
- J1 pad 2: VOLUME_2 -> GND
- J1 pad 3: GND -> VOLUME_2
- J10 pad 3: I2C1_SDA -> I2C1_SCL
- J10 pad 4: I2C1_SCL -> I2C1_SDA
- J11 pad 2: VOLUME_4 -> GND
- J11 pad 3: GND -> VOLUME_4
- J12 pad 3: UART1_RX -> UART1_TX
- J12 pad 4: UART1_TX -> UART1_RX
- J14 pad 1: BUTTON4 -> BUTTON1
- J14 pad 2: BUTTON3 -> BUTTON2
- J14 pad 3: BUTTON2 -> BUTTON3
- J14 pad 4: BUTTON1 -> BUTTON4
- J19 pad 2: RIGHT_JOYSTICK_IN1 -> GND
- J19 pad 3: GND -> RIGHT_JOYSTICK_IN1
- J20 pad 1: unconnected-(J20-Pin_1-Pad1) -> PB1
- J20 pad 2: unconnected-(J20-Pin_2-Pad2) -> GND
- J21 pad 1: unconnected-(J21-Pin_1-Pad1) -> PB3
- J21 pad 2: unconnected-(J21-Pin_2-Pad2) -> GND
- J22 pad 1: unconnected-(J22-Pin_1-Pad1) -> PC13
- J22 pad 2: unconnected-(J22-Pin_2-Pad2) -> GND
- J3 pad 2: LEFT_JOYSTICK_IN1 -> GND
- J3 pad 3: GND -> LEFT_JOYSTICK_IN1
- J4 pad 2: LEFT_JOYSTICK_IN2 -> GND
- J4 pad 3: GND -> LEFT_JOYSTICK_IN2
- J5 pad 2: RIGHT_JOYSTICK_IN2 -> GND
- J5 pad 3: GND -> RIGHT_JOYSTICK_IN2
- J6 pad 1: unconnected-(J6-Pin_1-Pad1) -> PB12
- J6 pad 2: unconnected-(J6-Pin_2-Pad2) -> GND
- J8 pad 2: VOLUME_1 -> GND
- J8 pad 3: GND -> VOLUME_1
- J9 pad 2: VOLUME_3 -> GND
- J9 pad 3: GND -> VOLUME_3
- U1 pad 19: unconnected-(U1-PB1-Pad19) -> PB1
- U1 pad 2: unconnected-(U1-PC13-Pad2) -> PC13
- U1 pad 22: NRF24_IRQ -> NRF24_CS
- U1 pad 25: NRF24_CS -> PB12
- U1 pad 38: unconnected-(U1-PA15-Pad38) -> NRF24_IRQ
- U1 pad 39: unconnected-(U1-PB3-Pad39) -> PB3
Routing:
- net PB12: track 0.00 -> 43.6 mm, vias 0 -> 1
- net PB3: track 0.00 -> 39.2 mm, vias 0 -> 2
- net +3V3: track 205.0 -> 240.6 mm, vias 4 -> 8
- net PB1: track 0.00 -> 27.0 mm, vias 0 -> 1
- net STM32_RESET: track 41.7 -> 66.9 mm
- net PC13: track 0.00 -> 16.7 mm
- net Net-(U1-BOOT0): track 20.6 -> 7.06 mm, vias 2 -> 0
- net BUTTON3: track 13.3 -> 23.0 mm
- net BUTTON4: track 16.1 -> 25.1 mm
- net RIGHT_JOYSTICK_IN1: track 26.9 -> 35.6 mm
- net NRF24_IRQ: track 21.2 -> 29.7 mm
- net PB10: track 35.5 -> 43.1 mm, vias 2 -> 1
- net 5V_DEBUGGER: track 56.7 -> 64.1 mm
- net NRF24_MISO: track 19.7 -> 26.8 mm
- net NRF24_CLK: track 20.1 -> 26.6 mm
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Other:
- board size 57 x 32 mm -> 62 x 37 mm
- board text added: "+"
- board text added: "-"
- board text added: "A0"
- board text added: "A1"
- board text added: "A3"
- board text added: "A4"
- board text added: "A5"
- board text added: "A6"
- board text added: "A7"
- board text added: "B1"
- board text added: "B10"
- board text added: "B12"
- board text added: "B2"
- board text added: "B3"
- board text added: "B4"
- board text added: "B5"
- board text added: "C13"
- board text added: "G"
- board text added: "MI"
- board text added: "MO"
- board text added: "OpenDrone Transmitter_F103_HW V2.0 Github: phonght32"
- board text added: "R1"
- board text added: "T1"
- board text removed: "LIN1"
- board text removed: "LIN2"
- board text removed: "OpenDrone Transmitter_F103_HW V1.0 Github: phonght32"
- board text removed: "RIN1"
- board text removed: "RIN2"
- board text removed: "RX1"
- board text removed: "SW1"
- board text removed: "SW2"
- board text removed: "SW3"
- board text removed: "SW4"
- board text removed: "TX1"
- board text removed: "VBAT"
- board text removed: "VOL1"
- board text removed: "VOL2"
- board text removed: "VOL3"
- board text removed: "VOL4"
