File: OpenDrone_Transmitter_F103_HW.kicad_pcb (KiCad board)
At the start: 2 copper layers, 62 x 37 mm, 87 parts, among them J1 Conn_01x03, J10 Conn_01x04, J11 Conn_01x03, J12 Conn_01x04, J13 Conn_01x02, J14 Conn_01x05, J15 Conn_01x02, J16 Conn_02x04_Odd_Even, J17 Conn_01x02, J18 Conn_01x02, J19 Conn_01x03, J2 Conn_01x05, J20 Conn_01x02, J21 Conn_01x02, J22 Conn_01x02, J23 Conn_01x08, J3 Conn_01x03, J4 Conn_01x03, J5 Conn_01x03, J6 Conn_01x02, J7 Conn_01x02, J8 Conn_01x03, J9 Conn_01x03, SW1 RESET, U1 STM32F103C8Tx, U2 AMS1117-3.3, U3 TPS54331, Y2 Crystal_GND24

Commit message: update text
Other:
- board text added: "A2"
Changed lines of the file:
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@@
 	)
 	(gr_text "3V3"
-		(at 168.3004 82.2706 0)
+		(at 168.151201 82.2706 0)
 		(layer "B.SilkS")
 		(effects
@@
 	)
 	(gr_text "GND"
-		(at 172.5676 83.4898 0)
+		(at 172.449999 83.4898 0)
 		(layer "B.SilkS")
 		(effects
@@
 		)
 	)
-	(gr_text "A3"
-		(at 168.3512 84.7852 0)
+	(gr_text "A0"
+		(at 167.484534 84.7852 0)
 		(layer "B.SilkS")
 		(effects
@@
 		)
 	)
-	(gr_text "A4"
-		(at 172.5676 84.7598 0)
+	(gr_text "A1"
+		(at 171.583333 84.7598 0)
 		(layer "B.SilkS")
 		(effects
@@
 	)
 	(gr_text "3V3"
-		(at 172.5168 82.2452 0)
+		(at 172.25 82.2452 0)
 		(layer "B.SilkS")
 		(effects
@@
 		)
 	)
-	(gr_text "A1"
+	(gr_text "A3"
 		(at 218.6178 82.296 0)
 		(layer "B.SilkS")
@@
 		)
 	)
-	(gr_text "A0"
+	(gr_text "A2"
 		(at 222.8342 82.2706 0)
 		(layer "B.SilkS")
